File: pcb/carte_embarque/carte_embarque.kicad_pcb (KiCad board)
At the start: 2 copper layers, 90 x 50 mm, 34 parts, among them J1 Conn_01x02, J2 Conn_01x02, J3 Conn_01x02, J4 Conn_01x02, Q1 NTD5865NLT4G, Q2 NTD5865NLT4G, U1 STM32L031, U2 XBee, U3 STEVAL-MKI176V1, U4 MIC4427

Commit message: petites evolutions sur PCB
Routing:
- net GND: vias 2 -> 5
- net GNDPWR: vias 3 -> 6
Changed lines of the file:
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@@
     (thickness 1.6)
     (drawings 7)
-    (tracks 326)
+    (tracks 333)
     (zones 0)
     (modules 34)
@@
     (visible_elements FFFFFF7F)
     (pcbplotparams
-      (layerselection 0x01000_ffffffff)
-      (usegerberextensions false)
+      (layerselection 0x0103c_ffffffff)
+      (usegerberextensions true)
       (usegerberattributes false)
       (usegerberadvancedattributes false)
       (creategerberjobfile false)
-      (excludeedgelayer false)
+      (excludeedgelayer true)
       (linewidth 0.100000)
       (plotframeref false)
@@
       (psa4output false)
       (plotreference true)
-      (plotvalue true)
+      (plotvalue false)
       (plotinvisibletext false)
       (padsonsilk false)
       (subtractmaskfromsilk false)
-      (outputformat 4)
+      (outputformat 1)
       (mirror false)
-      (drillshape 2)
+      (drillshape 0)
       (scaleselection 1)
       (outputdirectory "./"))
@@
     (effects (font (size 1.5 1.5) (thickness 0.3)))
   )
-  (gr_text "GEI 2019\n1.0" (at 129.53 100.005 90) (layer F.Cu)
+  (gr_text "GEI 2019\n1.0" (at 129.53 100.005 90) (layer F.SilkS)
     (effects (font (size 1.5 1.5) (thickness 0.3)))
   )
@@
   (segment (start 123.815 91.115) (end 123.815 93.655) (width 1) (layer B.Cu) (net 2))
   (segment (start 123.815 93.655) (end 123.18 94.29) (width 1) (layer B.Cu) (net 2))
-  (segment (start 123.18 94.29) (end 114.29 94.29) (width 1) (layer B.Cu) (net 2))
+  (segment (start 123.18 94.29) (end 116.195 94.29) (width 1) (layer B.Cu) (net 2))
   (segment (start 113.655 93.655) (end 113.655 91.115) (width 1) (layer B.Cu) (net 2))
   (segment (start 114.29 94.29) (end 113.655 93.655) (width 1) (layer B.Cu) (net 2))
+  (via (at 89.525 92.385) (size 1.3) (drill 0.7) (layers F.Cu B.Cu) (net 2))
+  (segment (start 116.195 94.29) (end 114.29 94.29) (width 1) (layer B.Cu) (net 2))
+  (via (at 116.195 94.29) (size 1.3) (drill 0.7) (layers F.Cu B.Cu) (net 2))
+  (via (at 114.925 80.955) (size 1.3) (drill 0.7) (layers F.Cu B.Cu) (net 2))
   (segment (start 103.8325 75.6575) (end 103.845 75.67) (width 1) (layer B.Cu) (net 3) (status 30))
   (segment (start 103.8325 75.6575) (end 103.845 75.67) (width 1) (layer F.Cu) (net 3) (status 30))
@@
   (segment (start 128.26 100.005) (end 126.99 98.735) (width 3) (layer B.Cu) (net 10))
   (segment (start 150.485 100.005) (end 128.26 100.005) (width 3) (layer B.Cu) (net 10))
+  (via (at 165.09 80.32) (size 1.3) (drill 0.7) (layers F.Cu B.Cu) (net 10))
+  (via (at 165.09 87.305) (size 1.3) (drill 0.7) (layers F.Cu B.Cu) (net 10))
+  (via (at 165.09 95.56) (size 1.3) (drill 0.7) (layers F.Cu B.Cu) (net 10))
   (segment (start 150.225 62.6975) (end 150.0675 62.54) (width 0.5) (layer F.Cu) (net 11) (status 30))
   (segment (start 150.225 65.96) (end 150.225 62.6975) (width 0.5) (layer F.Cu) (net 11) (status 30))
